Commit message: Collision enabled

File: src/my_robot_description/urdf/arm.xacro (robot description, xacro)
@@ -9,4 +9,10 @@
             <material name="grey" />
         </visual>
+        <collision>
+            <geometry>
+                <box size="0.4 0.4 0.1"/>
+            </geometry>
+            <origin xyz="0.0 0.0 0.05" rpy="0.0 0.0 0.0"/>
+        </collision>
     </link>
     <link name="shoulder_link">
@@ -18,4 +24,10 @@
             <material name="blue" />
         </visual>
+        <collision>
+            <geometry>
+                <cylinder radius="0.1" length="0.5"/>
+            </geometry>
+            <origin xyz="0 0 0.25" rpy="0 0 0" />
+        </collision>
     </link>
     <link name="arm_link">
@@ -27,4 +39,10 @@
             <material name="silver" />
         </visual>
+        <collision>
+            <geometry>
+                <cylinder radius="0.05" length="0.6"/>
+            </geometry>
+            <origin xyz="0 0 0.3" rpy="0 0 0" />
+        </collision>
     </link>
     <link name="elbow_link">
@@ -36,4 +54,10 @@
             <material name="blue" />
         </visual>
+        <collision>
+            <geometry>
+                <cylinder radius="0.05" length="0.1"/>
+            </geometry>
+            <origin xyz="0 0 0.05" rpy="0 0 0" />
+        </collision>
     </link>
     <link name="forearm_link">
@@ -45,4 +69,10 @@
             <material name="silver" />
         </visual>
+        <collision>
+            <geometry>
+                <cylinder radius="0.05" length="0.5"/>
+            </geometry>
+            <origin xyz="0 0 0.25" rpy="0 0 0" />
+        </collision>
     </link>
     <link name="wrist_link">
@@ -54,4 +84,10 @@
             <material name="blue" />
         </visual>
+        <collision>
+            <geometry>
+                <box size="0.1 0.1 0.05"/>
+            </geometry>
+            <origin xyz="0.0 0.0 0.025" rpy="0.0 0.0 0.0"/>
+        </collision>
     </link>
     <link name="hand_link">
@@ -63,4 +99,10 @@
             <material name="silver" />
         </visual>
+        <collision>
+            <geometry>
+                <box size="0.1 0.1 0.02"/>
+            </geometry>
+            <origin xyz="0.0 0.0 0.01" rpy="0.0 0.0 0.0"/>
+        </collision>
     </link>
     <link name="tool_link">
